File: Adapters/Adapters for programming/ATTiny85/ATTiny85.sch (KiCad schematic (older format))
At the start: 2 parts, among them U2 ATtiny85

Commit message: Signed all the boards, and re-generated the Gerber files
Parts:
- A1: footprint ArduinoUnoMultiProgrammerAdapters:Arduino-UNO-R3-Shield -> ArduinoUnoMultiProgrammerAdapters:Arduino_UNO_R3_Headers
Changed lines of the file:
@@
 F 0 "A1" H 5600 4931 50  0000 C CNN
 F 1 "Arduino_UNO_R3" H 5600 4840 50  0001 C CNN
-F 2 "ArduinoUnoMultiProgrammerAdapters:Arduino-UNO-R3-Shield" H 5600 3750 50  0001 C CIN
+F 2 "ArduinoUnoMultiProgrammerAdapters:Arduino_UNO_R3_Headers" H 5600 3750 50  0001 C CIN
 F 3 "https://www.arduino.cc/en/Main/arduinoBoardUno" H 5600 3750 50  0001 C CNN
 	1    5600 3750
