File: Adapters/Adapters for programming/Esp07/ESP-07.sch (KiCad schematic (older format))
At the start: 4 parts, among them U1 ESP-07

Commit message: Fixed error in ESP breadboard adapter footprint, updated the schema to wire the for the new layout. Updated the ESP flashing adapter.
Parts:
- A1: footprint ArduinoUnoMultiProgrammerAdapters:Arduino-UNO-R3-Shield -> ArduinoUnoMultiProgrammerAdapters:Arduino_UNO_R3_Headers
- U1: footprint ArduinoUnoMultiProgrammerAdapters:ESP-07-Socket -> ArduinoUnoMultiProgrammerAdapters:ESP07BreaboardSocket
Changed lines of the file:
@@
 F 0 "U1" H 3250 4681 50  0000 C CNN
 F 1 "ESP-07" H 3250 4590 50  0000 C CNN
-F 2 "ArduinoUnoMultiProgrammerAdapters:ESP-07-Socket" H 3250 3700 50  0001 C CNN
+F 2 "ArduinoUnoMultiProgrammerAdapters:ESP07BreaboardSocket" H 3250 3700 50  0001 C CNN
 F 3 "http://wiki.ai-thinker.com/_media/esp8266/esp8266_series_modules_user_manual_v1.1.pdf" H 2900 3800 50  0001 C CNN
 	1    3250 3700
@@
 F 0 "A1" H 6400 4881 50  0000 C CNN
 F 1 "Arduino_UNO_R3" H 6900 4800 50  0000 C CNN
-F 2 "ArduinoUnoMultiProgrammerAdapters:Arduino-UNO-R3-Shield" H 6400 3700 50  0001 C CIN
+F 2 "ArduinoUnoMultiProgrammerAdapters:Arduino_UNO_R3_Headers" H 6400 3700 50  0001 C CIN
 F 3 "https://www.arduino.cc/en/Main/arduinoBoardUno" H 6400 3700 50  0001 C CNN
 	1    6400 3700

Commit message: Fixed schematic for ESP adapter and regenerated Gerber files
Connections:
- net GND: now also U1.12 (GPIO0)
- no-connect marks 35 -> 34
Changed lines of the file:
@@
 NoConn ~ 2650 3500
 NoConn ~ 2650 3100
-NoConn ~ 3850 3100
 NoConn ~ 3850 3300
 NoConn ~ 3850 3500
@@
 	1    0    0    -1
 $EndComp
+Wire Wire Line
+	4550 4000 4550 3100
+Connection ~ 4550 4000
+Wire Wire Line
+	4550 3100 3850 3100
 $EndSCHEMATC
